File: main.kicad_pcb (KiCad board)
At the start: 4 copper layers, 40 x 35.2 mm, 25 parts, among them IC1 FR9888SPGTR, J1 LOAD+, J2 LOAD+, J3 LOAD+, J4 LOAD-, J5 support, U1 LM358

Commit message: v1
Parts:
- added REF**: R_1206_3216Metric, Resistor_SMD:R_1206_3216Metric, B.Cu at (154.4, 124.7)
- D2: footprint Diode_SMD:D_SOD-80C -> !my-kicad-library:D_4148_SMD
- moved C7 9.92 mm to (151.9, 123.2), turned to 90 degrees
- moved R3 7.70 mm to (144.5, 117.3), turned to 180 degrees
- moved D2 7.23 mm to (140.5, 120.1), turned to 180 degrees
- moved R2 5.64 mm to (148.8, 117.3), turned to 0 degrees
- moved R1 3.56 mm to (145.0, 124.9), turned to 180 degrees
- moved H3 2.13 mm to (131.3, 137.9)
- moved J5 1.62 mm to (149.9, 114.0)
- moved J4 1.17 mm to (156.0, 138.9)
- moved H1 1.15 mm to (162.6, 136.1)
- moved H2 0.82 mm to (145.3, 110.0)
- moved J3 0.55 mm to (132.3, 132.5)
- moved U1 0.51 mm to (146.8, 121.2)
- moved C2 0.45 mm to (148.6, 127.0)
Connections:
- U1 pad 1: Net-(D2-Pad2) -> Net-(U1-Pad1)
- U1 pad 2: Net-(R2-Pad1) -> Net-(U1-Pad1)
- U1 pad 3: LOAD- -> GND
- U1 pad 5: GND -> LOAD-
- U1 pad 6: Net-(U1-Pad6) -> Net-(R2-Pad1)
- U1 pad 7: Net-(U1-Pad6) -> Net-(D2-Pad2)
Routing:
- net V_IN: track 25.1 -> 55.4 mm
- net Net-(R2-Pad1): track 4.18 -> 18.4 mm
- net LOAD-: track 46.6 -> 38.3 mm, vias 0 -> 2
- net Feedback: track 17.9 -> 9.68 mm
- net GND: track 48.6 -> 54.3 mm
- net Net-(U1-Pad6): track 2.63 -> 0.00 mm
- net Net-(IC1-Pad7): track 4.06 -> 2.13 mm
- net Net-(U1-Pad1): track 0.00 -> 1.27 mm
- net Net-(D2-Pad2): track 5.71 -> 6.23 mm

Commit message: last fixes
Parts:
- C1: value 100n -> 100nF
- R2: value 560 -> 820
- R3: value 43k -> 30k
Other:
- board text added: "0"
Changed lines of the file:
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@@
     (fp_line (start -0.883605 -1.3375) (end -0.883605 -0.8375) (layer "F.Fab") (width 0.1))
     (fp_circle (center 1 0) (end 3.5 0) (layer "F.Fab") (width 0.1) (fill none))
-    (pad "1" thru_hole rect locked (at 0 0 90) (size 1.6 1.6) (drill 0.8) (layers *.Cu *.Mask)
+    (pad "1" thru_hole rect (at 0 0 90) (size 1.6 1.6) (drill 0.8) (layers *.Cu *.Mask)
       (net 8 "LOAD+") (pintype "passive"))
-    (pad "2" thru_hole circle locked (at 2 0 90) (size 1.6 1.6) (drill 0.8) (layers *.Cu *.Mask)
+    (pad "2" thru_hole circle (at 2 0 90) (size 1.6 1.6) (drill 0.8) (layers *.Cu *.Mask)
       (net 2 "GND") (pintype "passive"))
     (model "${KICAD6_3DMODEL_DIR}/Capacitor_THT.3dshapes/CP_Radial_D5.0mm_P2.00mm.wrl"
@@
     (fp_line (start -1.443972 -1.3735) (end -0.813972 -1.3735) (layer "F.Fab") (width 0.1))
     (fp_circle (center 1.25 0) (end 4.4 0) (layer "F.Fab") (width 0.1) (fill none))
-    (pad "1" thru_hole rect locked (at 0 0) (size 1.6 1.6) (drill 0.8) (layers *.Cu *.Mask)
+    (pad "1" thru_hole rect (at 0 0) (size 1.6 1.6) (drill 0.8) (layers *.Cu *.Mask)
       (net 1 "V_IN") (pintype "passive"))
-    (pad "2" thru_hole circle locked (at 2.5 0) (size 1.6 1.6) (drill 0.8) (layers *.Cu *.Mask)
+    (pad "2" thru_hole circle (at 2.5 0) (size 1.6 1.6) (drill 0.8) (layers *.Cu *.Mask)
       (net 2 "GND") (pintype "passive"))
     (model "${KICAD6_3DMODEL_DIR}/Capacitor_THT.3dshapes/CP_Radial_D6.3mm_P2.50mm.wrl"
@@
       (effects (font (size 1 1) (thickness 0.15)) (justify mirror))
     )
-    (fp_text value "100nF" (at 4.630608 -0.013169) (layer "B.Fab")
+    (fp_text value "100nF" (at -0.053463 1.780849) (layer "B.Fab")
       (effects (font (size 1 1) (thickness 0.15)) (justify mirror))
     )
@@
       (effects (font (size 1 1) (thickness 0.15)) (justify mirror))
     )
-    (fp_text value "FR9888SPGTR" (at 0 -3.4 90) (layer "B.Fab") hide
+    (fp_text value "FR9888SPGTR" (at 0.55375 -8.255 180) (layer "B.Fab")
       (effects (font (size 1 1) (thickness 0.15)) (justify mirror))
     )
@@
       (effects (font (size 1 1) (thickness 0.15)) (justify mirror))
     )
-    (fp_text value "100n" (at 0 -1.85 90) (layer "B.Fab")
+    (fp_text value "100n" (at 3.556 0 90) (layer "B.Fab")
       (effects (font (size 1 1) (thickness 0.15)) (justify mirror))
     )
@@
       (effects (font (size 1 1) (thickness 0.15)) (justify mirror))
     )
-    (fp_text value "91k" (at 0 -1.65) (layer "B.Fab")
+    (fp_text value "91k" (at 3.048 0) (layer "B.Fab")
       (effects (font (size 1 1) (thickness 0.15)) (justify mirror))
     )
@@
       (effects (font (size 1 1) (thickness 0.15)) (justify mirror))
     )
-    (fp_text value "MBRA340T3G" (at 0 -2.6) (layer "B.Fab")
-      (effects (font (size 1 1) (thickness 0.15)) (justify mirror))
-    )
-    (fp_text user "${REFERENCE}" (at 0 2.5) (layer "B.Fab")
+    (fp_text value "MBRA340T3G" (at 0.032 3.81) (layer "B.Fab")
+      (effects (font (size 1 1) (thickness 0.15)) (justify mirror))
+    )
+    (fp_text user "${REFERENCE}" (at 0.54 -2.54) (layer "B.Fab")
       (effects (font (size 1 1) (thickness 0.15)) (justify mirror))
     )
@@
       (effects (font (size 1 1) (thickness 0.15)) (justify mirror))
     )
-    (fp_text value "LM358" (at 0 -3.4) (layer "B.Fab")
-      (effects (font (size 1 1) (thickness 0.15)) (justify mirror))
-    )
-    (fp_text user "${REFERENCE}" (at 0 0) (layer "B.Fab")
+    (fp_text value "LM358" (at 0 0 90) (layer "B.Fab")
+      (effects (font (size 1 1) (thickness 0.15)) (justify mirror))
+    )
+    (fp_text user "${REFERENCE}" (at 0 0) (layer "B.Fab") hide
       (effects (font (size 0.98 0.98) (thickness 0.15)) (justify mirror))
     )
@@
     )
   )
-  (footprint "!my-kicad-library:SolderWire-slot" (layer "B.Cu")
+  (footprint "!my-kicad-library:SolderWire-slot" locked (layer "B.Cu")
     (at 132.334 132.5 180)
     (descr "Soldered wire connection, for a single 0.1 mm² wire, basic insulation, conductor diameter 0.4mm, outer diameter 1mm, size source Multi-Contact FLEXI-E 0.1 (https://ec.staubli.com/AcroFiles/Catalogues/TM_Cab-Main-11014119_(en)_hi.pdf), bend radius 3 times outer diameter, generated with kicad-footprint-generator")
@@
     (property "Sheetfile" "main.kicad_sch")
     (property "Sheetname" "")
-    (attr exclude_from_pos_files)
     (fp_text reference "J3" (at 0 4) (layer "B.SilkS") hide
       (effects (font (size 1 1) (thickness 0.15)) (justify mirror))
@@
     (fp_rect (start -2 2) (end 2 -2) (layer "B.CrtYd") (width 0.12) (fill none))
     (fp_rect (start -1.778 1.778) (end 1.778 -1.778) (layer "B.Fab") (width 0.1) (fill none))
-    (pad "1" thru_hole roundrect (at 0 0 20) (size 3 3.5) (drill oval 1 3) (layers *.Cu *.Mask) (roundrect_rratio 0.25)
+    (pad "1" thru_hole roundrect locked (at 0 0 20) (size 3 3.5) (drill oval 1 3) (layers *.Cu *.Mask) (roundrect_rratio 0.25)
       (net 8 "LOAD+") (pinfunction "Pin_1") (pintype "passive"))
     (model "${KICAD6_3DMODEL_DIR}/Connector_Wire.3dshapes/SolderWire-0.1sqmm_1x01_D0.4mm_OD1mm.wrl"
@@
       (effects (font (size 1 1) (thickness 0.15)) (justify mirror))
     )
-    (fp_text value "100k" (at 3.043561 -3.084705) (layer "B.Fab")
+    (fp_text value "100k" (at 2.794 0.151616) (layer "B.Fab")
       (effects (font (size 1 1) (thickness 0.15)) (justify mirror))
     )
@@
       (effects (font (size 1 1) (thickness 0.15)) (justify mirror))
     )
-    (fp_text value "43k" (at -3.922313 -0.017671) (layer "B.Fab")
+    (fp_text value "30k" (at 0 1.524) (layer "B.Fab")
       (effects (font (size 1 1) (thickness 0.15)) (justify mirror))
     )
@@
       (effects (font (size 1 1) (thickness 0.15)) (justify mirror))
     )
-    (fp_text value "100n" (at -0.185078 4.240158) (layer "B.Fab")
+    (fp_text value "100nF" (at 0 -2.032) (layer "B.Fab")
       (effects (font (size 1 1) (thickness 0.15)) (justify mirror))
     )
@@
       (effects (font (size 1 1) (thickness 0.15)) (justify mirror))
     )
-    (fp_text value "100uH" (at 0 -4.5) (layer "B.Fab")
+    (fp_text value "100uH" (at 0 -1.61) (layer "B.Fab")
       (effects (font (size 1 1) (thickness 0.15)) (justify mirror))
     )
@@
       (effects (font (size 0.70104 0.70104) (thickness 0.14986)) (justify mirror))
     )
-    (fp_text value "1N4148" (at 0.0254 -1.397) (layer "B.SilkS") hide
+    (fp_text value "1N4148" (at 4.870951 -0.00237) (layer "B.Fab")
       (effects (font (size 0.70104 0.70104) (thickness 0.14986)) (justify mirror))
     )
@@
       (effects (font (size 1 1) (thickness 0.15)) (justify mirror))
     )
-    (fp_text value "R_1206_3216Metric" (at 0 -1.82 90) (layer "B.Fab")
-      (effects (font (size 1 1) (thickness 0.15)) (justify mirror))
-    )
-    (fp_text user "${REFERENCE}" (at 0 0 90) (layer "B.Fab")
+    (fp_text value "R_1206_3216Metric" (at 0 -1.82 90) (layer "B.Fab") hide
+      (effects (font (size 1 1) (thickness 0.15)) (justify mirror))
+    )
+    (fp_text user "${REFERENCE}" (at 0 0 90) (layer "B.Fab") hide
       (effects (font (size 0.8 0.8) (thickness 0.12)) (justify mirror))
     )
@@
       (effects (font (size 1 1) (thickness 0.15)) (justify mirror))
     )
-    (fp_text value "100m" (at 0 -2.62) (layer "B.Fab")
+    (fp_text value "100m" (at 0.254 -2.286) (layer "B.Fab")
       (effects (font (size 1 1) (thickness 0.15)) (justify mirror))
     )
@@
       (effects (font (size 1 1) (thickness 0.15)) (justify mirror))
     )
-    (fp_text value "15k" (at 0 -1.65) (layer "B.Fab")
+    (fp_text value "15k" (at -3.051904 0.039372) (layer "B.Fab")
       (effects (font (size 1 1) (thickness 0.15)) (justify mirror))
     )
@@
     (fp_line (start -1.9 1.65) (end -1.9 -1.65) (layer "B.CrtYd") (width 0.05))
     (fp_circle (center 0 0) (end 1.15 0) (layer "B.Fab") (width 0.1) (fill none))
-    (pad "1" thru_hole roundrect locked (at 0 0 180) (size 2.3 2.3) (drill 1.1) (layers *.Cu *.Mask) (roundrect_rratio 0.108696)
+    (pad "1" thru_hole roundrect (at 0 0 180) (size 2.3 2.3) (drill 1.1) (layers *.Cu *.Mask) (roundrect_rratio 0.108696)
       (net 2 "GND") (pinfunction "Pin_1") (pintype "passive"))
     (model "${KICAD6_3DMODEL_DIR}/Connector_Wire.3dshapes/SolderWire-0.5sqmm_1x01_D0.9mm_OD2.3mm.wrl"
@@
       (effects (font (size 1 1) (thickness 0.15)) (justify mirror))
     )
-    (fp_text value "560" (at 3.421639 -0.127115) (layer "B.Fab")
+    (fp_text value "820" (at 0.254 -1.524) (layer "B.Fab")
       (effects (font (size 1 1) (thickness 0.15)) (justify mirror))
     )
@@
   (gr_text "LOAD+" (at 129.54 135.382) (layer "B.SilkS")
     (effects (font (size 0.8128 0.8128) (thickness 0.1524)) (justify mirror))
+  )
+  (gr_text "0" (at 154.432 124.714) (layer "B.Fab")
+    (effects (font (size 1 1) (thickness 0.15)) (justify mirror))
   )
   (segment (start 156.161 124.665) (end 156.972 125.476) (width 0.6) (layer "B.Cu") (net 1))
@@
   (segment (start 142.31112 117.68138) (end 142.494 117.4985) (width 0.6) (layer "B.Cu") (net 15))
   (segment (start 142.43812 120.523) (end 142.31112 120.396) (width 0.6) (layer "B.Cu") (net 15))
-  (zone (net 0) (net_name "") (layer "B.Cu") (hatch edge 0.508)
-    (connect_pads (clearance 0))
-    (min_thickness 0.254)
-    (keepout (tracks allowed) (vias allowed) (pads allowed ) (copperpour not_allowed) (footprints allowed))
-    (fill (thermal_gap 0.508) (thermal_bridge_width 0.508))
-    (polygon
-      (pts
-        (xy 142.08 141.224)
-        (xy 133.74 141.224)
-        (xy 133.740001 133.560548)
-        (xy 142.080001 133.560548)
-      )
-    )
-  )
 )
