File: main.kicad_sch (KiCad schematic)
At the start: 25 parts, among them IC1 FR9888SPGTR, J1 LOAD+, J2 LOAD+, J3 LOAD+, J4 LOAD-, J5 support, U1 LM358

Commit message: v1
Parts:
- D2: footprint Diode_SMD:D_SOD-80C -> !my-kicad-library:D_4148_SMD
Connections:
- net GND: now also U1.3 (+); no longer U1.5 (+)
- net LOAD-: now also U1.5 (+); no longer U1.3 (+)
- net at D2.2 (A), R3.2: now also U1.7; no longer U1.1
- net at R2.1, R3.1: now also U1.6 (-); no longer U1.2 (-)
- new net: U1.1, U1.2 (-)
Changed lines of the file:
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@@
     (property "Reference" "D2" (id 0) (at 149.86 130.0185 0))
     (property "Value" "1N4148" (id 1) (at 149.86 132.7936 0))
-    (property "Footprint" "Diode_SMD:D_SOD-80C" (id 2) (at 149.86 130.81 0)
+    (property "Footprint" "!my-kicad-library:D_4148_SMD" (id 2) (at 149.86 130.81 0)
       (effects (font (size 1.27 1.27)) hide)
     )
@@
     (pin "2")
   )
-  (symbol (lib_id "Amplifier_Operational:LM358") (at 48.26 139.065 0) (unit 2)
+  (symbol (lib_id "Amplifier_Operational:LM358") (at 48.26 139.065 0) (unit 1)
     (in_bom yes) (on_board yes) (fields_autoplaced)
     (property "Reference" "U1" (id 0) (at 48.26 130.0185 0))
@@
       (effects (font (size 1.27 1.27)) hide)
     )
-    (pin "5")
-    (pin "6")
-    (pin "7")
+    (pin "1")
+    (pin "2")
+    (pin "3")
   )
   (symbol (lib_id "Device:C") (at 139.7 55.88 270) (unit 1)
@@
     (pin "1")
   )
-  (symbol (lib_id "Amplifier_Operational:LM358") (at 132.715 135.255 0) (unit 1)
+  (symbol (lib_id "Amplifier_Operational:LM358") (at 132.715 135.255 0) (unit 2)
     (in_bom yes) (on_board yes) (fields_autoplaced)
     (property "Reference" "U1" (id 0) (at 132.715 126.2085 0))
@@
       (effects (font (size 1.27 1.27)) hide)
     )
-    (pin "1")
-    (pin "2")
-    (pin "3")
+    (pin "5")
+    (pin "6")
+    (pin "7")
   )
   (symbol (lib_id "Device:C") (at 189.23 86.995 0) (unit 1)
@@
     )
     (path "/31518452-8dcd-4719-9aa4-aad4159920e6"
-      (reference "D2") (unit 1) (value "1N4148") (footprint "Diode_SMD:D_SOD-80C")
+      (reference "D2") (unit 1) (value "1N4148") (footprint "!my-kicad-library:D_4148_SMD")
     )
     (path "/42bcded6-6802-4b1c-a9a7-30a9314a5805"
@@
       (reference "R6") (unit 1) (value "15k") (footprint "Resistor_SMD:R_0805_2012Metric")
     )
+    (path "/31a27a84-3176-4648-b7d9-e64c84d02aba"
+      (reference "U1") (unit 1) (value "LM358") (footprint "Package_SO:SOIC-8_3.9x4.9mm_P1.27mm")
+    )
     (path "/ba156237-0f7a-4fb9-8f50-dad0b83870b9"
-      (reference "U1") (unit 1) (value "LM358") (footprint "Package_SO:SOIC-8_3.9x4.9mm_P1.27mm")
-    )
-    (path "/31a27a84-3176-4648-b7d9-e64c84d02aba"
       (reference "U1") (unit 2) (value "LM358") (footprint "Package_SO:SOIC-8_3.9x4.9mm_P1.27mm")
     )

Commit message: last fixes
Parts:
- C1: value 100n -> 100nF
- R2: value 560 -> 820
- R3: value 43k -> 30k
Other:
- note added: "0.55V @ 25C 0.45 @ 60C"
- note added: "input offset ±1mv"
- note added: "target -> 0.925V ± 0.25"
- note added: "trimmed/measured value"
- note removed: "0.925V"
Changed lines of the file:
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@@
+    (effects (font (size 1.27 1.27)) (justify left bottom))
+  )
+  (text "0.55V @ 25C\n0.45 @ 60C" (at 143.51 128.27 0)
     (effects (font (size 1.27 1.27)) (justify left bottom))
   )
@@
     (effects (font (size 1.27 1.27)) (justify left bottom))
   )
-  (text "0.925V\n" (at 159.385 133.35 0)
+  (text "target -> 0.925V ± 0.25\n" (at 159.385 133.35 0)
     (effects (font (size 1.27 1.27)) (justify left bottom))
+  )
+  (text "trimmed/measured value" (at 133.985 149.225 0)
+    (effects (font (size 1.27 1.27)) (justify left bottom))
+  )
+  (text "input offset ±1mv" (at 123.825 127 180)
+    (effects (font (size 1.27 1.27)) (justify right bottom))
   )
   (global_label "LOAD+" (shape input) (at 219.71 70.485 0) (fields_autoplaced)
@@
       (effects (font (size 1.27 1.27)) (justify left))
     )
-    (property "Value" "100n" (id 1) (at 107.315 86.995 0)
+    (property "Value" "100nF" (id 1) (at 107.315 86.995 0)
       (effects (font (size 1.27 1.27)) (justify left))
     )
@@
       (effects (font (size 1.27 1.27)) (justify left))
     )
-    (property "Value" "560" (id 1) (at 121.666 153.6316 0)
+    (property "Value" "820" (id 1) (at 121.666 153.6316 0)
       (effects (font (size 1.27 1.27)) (justify left))
     )
@@
     (in_bom yes) (on_board yes)
     (property "Reference" "R3" (id 0) (at 132.08 147.7199 90))
-    (property "Value" "43k" (id 1) (at 132.08 142.875 90))
+    (property "Value" "30k" (id 1) (at 132.08 142.875 90))
     (property "Footprint" "Resistor_SMD:R_0805_2012Metric" (id 2) (at 132.334 144.399 90)
       (effects (font (size 1.27 1.27)) hide)
@@
     )
     (path "/d1a9be32-38ba-44e6-bc35-f031541ab1fe"
-      (reference "C1") (unit 1) (value "100n") (footprint "Capacitor_SMD:C_1206_3216Metric")
+      (reference "C1") (unit 1) (value "100nF") (footprint "Capacitor_SMD:C_1206_3216Metric")
     )
     (path "/ed8a7f02-cf05-41d0-97b4-4388ef205e73"
@@
     )
     (path "/d2264311-a0a5-4f1b-8dc5-a05cce701216"
-      (reference "R2") (unit 1) (value "560") (footprint "Resistor_SMD:R_0805_2012Metric")
+      (reference "R2") (unit 1) (value "820") (footprint "Resistor_SMD:R_0805_2012Metric")
     )
     (path "/fb35717a-3024-4748-8c92-07b62abc226c"
-      (reference "R3") (unit 1) (value "43k") (footprint "Resistor_SMD:R_0805_2012Metric")
+      (reference "R3") (unit 1) (value "30k") (footprint "Resistor_SMD:R_0805_2012Metric")
     )
     (path "/2a159d98-9515-4045-afd5-7789f8903188"
